File: maquiavelo/maquiavelo.kicad_pcb (KiCad board)
At the start: 2 copper layers, 80 x 90 mm, 21 parts, among them IC1 ArduinoProMini, J1 Conn_01x11, J2 Conn_01x02, J3 Conn_01x02, U1 DRIVER, U4 button, U5 SVL6180X, U6 SVL6180X, U7 SVL6180X

Commit message: gerbers
Parts:
- added P1: bateria1, MAKI:JST_XH_B02B-XH-A_02x2.50mm_Straight, F.Cu at (72.4, 59.7)
- added P2: bateria2, MAKI:JST_XH_B02B-XH-A_02x2.50mm_Straight, F.Cu at (108.0, 59.7)
- G***: moved to B.Cu
- moved G*** 52.1 mm to (66.0, 73.7), turned to 180 degrees
- moved J3 2.54 mm to (106.7, 73.7)
- moved J2 1.80 mm to (76.2, 73.7)
- moved U4 1.78 mm to (87.7, 58.4)
Routing:
- net +5V: track 175.4 -> 99.7 mm, vias 2 -> 3
- net GND: track 177.1 -> 111.5 mm
- net +7.5V: track 46.2 -> 107.0 mm, vias 1 -> 3
- net Net-(P1-Pad2): track 0.00 -> 33.1 mm
- net /MI: track 52.9 -> 82.0 mm, vias 0 -> 1
- net /MD: track 60.1 -> 84.4 mm
- net /MD2: track 75.0 -> 93.4 mm, vias 3 -> 1
- net /MI2: track 51.3 -> 64.1 mm, vias 0 -> 1
- net /Q1: track 48.4 -> 54.0 mm
- net /A2: track 82.7 -> 88.0 mm
- net /PWMA: track 52.0 -> 56.7 mm
- net Net-(R1-Pad1): track 62.0 -> 64.6 mm
- net /SCL: track 124.1 -> 126.5 mm
- net /A1: track 58.4 -> 56.4 mm, vias 0 -> 2
- net /Q0: track 79.3 -> 81.3 mm
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Other:
- net class power added: clearance 0.2, trace_width 0.8, via_dia 1, via_drill 0.6
